Commit message: Added the lidar frame and link to nomad3.urdf.xacro.

File: nomad/models/nomad3.urdf.xacro (robot description, xacro)
@@ -19,4 +19,12 @@
     <xacro:property name="wheelTrack"     value="0.307" />
     <xacro:property name="axleHeight"     value="${wheelRadius}" />
+    <!--
+	 The definitions for the lidar.
+	 -->
+    <xacro:property name="lidarLength"    value="0.085" />
+    <xacro:property name="lidarRadius"    value="0.065" />
+    <xacro:property name="lidarOriginX"   value="0.0" />
+    <xacro:property name="lidarOriginY"   value="0.0" />
+    <xacro:property name="lidarOriginZ"   value="0.333" />
     <link name="base_link">
         <visual>
@@ -56,3 +64,16 @@
         </visual>
     </link>
+    <joint name="base_link_to_lidar" type="fixed">
+        <parent link="base_link"/>
+        <child link="lidar"/>
+        <origin xyz="${lidarOriginX} ${lidarOriginY} ${lidarOriginZ}"/>
+    </joint>
+    <link name="lidar">
+        <visual>
+            <origin xyz="0 0 0" rpy="0 0 0" />
+            <geometry>
+                <cylinder length="${lidarLength}" radius="${lidarRadius}" />
+            </geometry>
+        </visual>
+    </link>
 </robot>

Commit message: Added ultrasonic rangefinder frames to nomad3.urdf.xacro

File: nomad/models/nomad3.urdf.xacro (robot description, xacro)
@@ -27,4 +27,15 @@
     <xacro:property name="lidarOriginY"   value="0.0" />
     <xacro:property name="lidarOriginZ"   value="0.333" />
+    <!--
+	 The definitions for the ultrasonic rangefinders.
+	 -->
+    <xacro:property name="ultraLength"    value="0.020" />
+    <xacro:property name="ultraRadius"    value="0.008" />
+    <xacro:property name="ultraOriginXF"  value="0.055" />
+    <xacro:property name="ultraOriginXB"  value="-0.330" />
+    <xacro:property name="ultraOriginY"   value="0.070" />
+    <xacro:property name="ultraOriginZ"   value="0.187" />
+    <xacro:property name="ultraUp"        value="-0.1" />
+    <xacro:property name="ultraOut"       value="0.05" />
     <link name="base_link">
         <visual>
@@ -77,3 +88,68 @@
         </visual>
     </link>
+    <joint name="base_link_to_range_lf" type="fixed">
+        <parent link="base_link"/>
+        <child link="range_left_front"/>
+        <origin
+            xyz="${ultraOriginXF} ${ultraOriginY} ${ultraOriginZ}"
+            rpy="0 ${ultraUp} ${ultraOut}"
+            />
+    </joint>
+    <link name="range_left_front">
+        <visual>
+            <origin xyz="0 0 0"
+                />
+            <geometry>
+                <cylinder length="${ultraLength}" radius="${ultraRadius}" />
+            </geometry>
+        </visual>
+    </link>
+    <joint name="base_link_to_range_rf" type="fixed">
+        <parent link="base_link"/>
+        <child link="range_right_front"/>
+        <origin
+            xyz="${ultraOriginXF} -${ultraOriginY} ${ultraOriginZ}"
+            rpy="0 ${ultraUp} -${ultraOut}"
+            />
+    </joint>
+    <link name="range_right_front">
+        <visual>
+            <origin xyz="0 0 0" />
+            <geometry>
+                <cylinder length="${ultraLength}" radius="${ultraRadius}" />
+            </geometry>
+        </visual>
+    </link>
+    <joint name="base_link_to_range_lr" type="fixed">
+        <parent link="base_link"/>
+        <child link="range_left_rear"/>
+        <origin
+            xyz="${ultraOriginXB} ${ultraOriginY} ${ultraOriginZ}"
+            rpy="0 ${ultraUp} ${3.14-ultraOut}"
+            />
+    </joint>
+    <link name="range_left_rear">
+        <visual>
+            <origin xyz="0 0 0" />
+            <geometry>
+                <cylinder length="${ultraLength}" radius="${ultraRadius}" />
+            </geometry>
+        </visual>
+    </link>
+    <joint name="base_link_to_range_rr" type="fixed">
+        <parent link="base_link"/>
+        <child link="range_right_rear"/>
+        <origin
+            xyz="${ultraOriginXB} -${ultraOriginY} ${ultraOriginZ}"
+            rpy="0 ${ultraUp} ${3.14+ultraOut}"
+            />
+    </joint>
+    <link name="range_right_rear">
+        <visual>
+            <origin xyz="0 0 0" />
+            <geometry>
+                <cylinder length="${ultraLength}" radius="${ultraRadius}" />
+            </geometry>
+        </visual>
+    </link>
 </robot>

Commit message: Added camera_front frame to nomad3.urdf.xacro.

File: nomad/models/nomad3.urdf.xacro (robot description, xacro)
@@ -9,7 +9,15 @@
     <xacro:property name="mainPadWidth"   value="0.203" />
     <xacro:property name="mainPadHeight"  value="0.013" />
-    <xacro:property name="mainPadOriginX" value="-0.139" />
-    <xacro:property name="mainPadOriginY" value="0.0" />
-    <xacro:property name="mainPadOriginZ" value="0.190" />
+    <xacro:property name="mainPadX" value="-0.139" />
+    <xacro:property name="mainPadY" value="0.0" />
+    <xacro:property name="mainPadZ" value="0.198" />
+    <!--
+	 The definitions for the cameras.
+	 -->
+    <xacro:property name="cameraRadius"   value="0.015" />
+    <xacro:property name="cameraLength"   value="0.030" />
+    <xacro:property name="cameraFX"       value="0.0" />
+    <xacro:property name="cameraFY"       value="0.0" />
+    <xacro:property name="cameraFZ"       value="0.026" />
     <!--
 	 The definitions for the wheels.
@@ -40,5 +48,5 @@
     <link name="base_link">
         <visual>
-            <origin xyz="${mainPadOriginX} ${mainPadOriginY} ${mainPadOriginZ}" rpy="0 0 0" />
+            <origin xyz="${mainPadX} ${mainPadY} ${mainPadZ}" rpy="0 0 0" />
             <geometry>
                 <box size="${mainPadLength} ${mainPadWidth} ${mainPadHeight}" />
@@ -153,3 +161,19 @@
         </visual>
     </link>
+    <joint name="base_link_to_camera_front" type="fixed">
+        <parent link="base_link"/>
+        <child link="camera_front"/>
+        <origin
+            xyz="${cameraFX} ${cameraFY} ${mainPadZ + cameraFZ}"
+            rpy="-1.57 0 -1.57"
+            />
+    </joint>
+    <link name="camera_front">
+        <visual>
+            <origin xyz="0 0 0" />
+            <geometry>
+                <cylinder length="${cameraLength}" radius="${cameraRadius}" />
+            </geometry>
+        </visual>
+    </link>
 </robot>

Commit message: Changes to many files to use laser frame instead of lidar frame, to add queue_size argument to Publisher calls, to add SLAM and map server and robot_pose_ekf and robot_state_publisher.

File: nomad/models/nomad3.urdf.xacro (robot description, xacro)
@@ -83,10 +83,10 @@
         </visual>
     </link>
-    <joint name="base_link_to_lidar" type="fixed">
+    <joint name="base_link_to_laser" type="fixed">
         <parent link="base_link"/>
-        <child link="lidar"/>
+        <child link="laser"/>
         <origin xyz="${lidarOriginX} ${lidarOriginY} ${lidarOriginZ}"/>
     </joint>
-    <link name="lidar">
+    <link name="laser">
         <visual>
             <origin xyz="0 0 0" rpy="0 0 0" />

Commit message: Removed ultrasonic rangefinders from the URDF model in nomad/models/nomad3.urdf.xacro

File: nomad/models/nomad3.urdf.xacro (robot description, xacro)
@@ -96,69 +96,4 @@
         </visual>
     </link>
-    <joint name="base_link_to_range_lf" type="fixed">
-        <parent link="base_link"/>
-        <child link="range_left_front"/>
-        <origin
-            xyz="${ultraOriginXF} ${ultraOriginY} ${ultraOriginZ}"
-            rpy="0 ${ultraUp} ${ultraOut}"
-            />
-    </joint>
-    <link name="range_left_front">
-        <visual>
-            <origin xyz="0 0 0"
-                />
-            <geometry>
-                <cylinder length="${ultraLength}" radius="${ultraRadius}" />
-            </geometry>
-        </visual>
-    </link>
-    <joint name="base_link_to_range_rf" type="fixed">
-        <parent link="base_link"/>
-        <child link="range_right_front"/>
-        <origin
-            xyz="${ultraOriginXF} -${ultraOriginY} ${ultraOriginZ}"
-            rpy="0 ${ultraUp} -${ultraOut}"
-            />
-    </joint>
-    <link name="range_right_front">
-        <visual>
-            <origin xyz="0 0 0" />
-            <geometry>
-                <cylinder length="${ultraLength}" radius="${ultraRadius}" />
-            </geometry>
-        </visual>
-    </link>
-    <joint name="base_link_to_range_lr" type="fixed">
-        <parent link="base_link"/>
-        <child link="range_left_rear"/>
-        <origin
-            xyz="${ultraOriginXB} ${ultraOriginY} ${ultraOriginZ}"
-            rpy="0 ${ultraUp} ${3.14-ultraOut}"
-            />
-    </joint>
-    <link name="range_left_rear">
-        <visual>
-            <origin xyz="0 0 0" />
-            <geometry>
-                <cylinder length="${ultraLength}" radius="${ultraRadius}" />
-            </geometry>
-        </visual>
-    </link>
-    <joint name="base_link_to_range_rr" type="fixed">
-        <parent link="base_link"/>
-        <child link="range_right_rear"/>
-        <origin
-            xyz="${ultraOriginXB} -${ultraOriginY} ${ultraOriginZ}"
-            rpy="0 ${ultraUp} ${3.14+ultraOut}"
-            />
-    </joint>
-    <link name="range_right_rear">
-        <visual>
-            <origin xyz="0 0 0" />
-            <geometry>
-                <cylinder length="${ultraLength}" radius="${ultraRadius}" />
-            </geometry>
-        </visual>
-    </link>
     <joint name="base_link_to_camera_front" type="fixed">
         <parent link="base_link"/>

Commit message: Changed wheel joints from continuous to fixed in nomad/models/nomad3.urdf.xacro

File: nomad/models/nomad3.urdf.xacro (robot description, xacro)
@@ -57,5 +57,5 @@
         </visual>
     </link>
-    <joint name="base_link_to_right_wheel" type="continuous">
+    <joint name="base_link_to_right_wheel" type="fixed">
         <parent link="base_link"/>
         <child link="right_wheel"/>
@@ -70,5 +70,5 @@
         </visual>
     </link>
-    <joint name="base_link_to_left_wheel" type="continuous">
+    <joint name="base_link_to_left_wheel" type="fixed">
         <parent link="base_link"/>
         <child link="left_wheel"/>

Commit message: Updated config/diff_baseController.xml and models/nomad3.urdf.xacro with mower prototype chassis parameters.

File: nomad/models/nomad3.urdf.xacro (robot description, xacro)
@@ -23,7 +23,7 @@
 	 The definitions for the wheels.
 	 -->
-    <xacro:property name="wheelRadius"    value="0.096" />
-    <xacro:property name="wheelWidth"     value="0.050" />
-    <xacro:property name="wheelTrack"     value="0.307" />
+    <xacro:property name="wheelRadius"    value="0.073" />
+    <xacro:property name="wheelWidth"     value="0.085" />
+    <xacro:property name="wheelTrack"     value="0.31" />
     <xacro:property name="axleHeight"     value="${wheelRadius}" />
     <!--
@@ -33,6 +33,6 @@
     <xacro:property name="lidarRadius"    value="0.065" />
     <xacro:property name="lidarOriginX"   value="0.0" />
-    <xacro:property name="lidarOriginY"   value="0.0" />
-    <xacro:property name="lidarOriginZ"   value="0.333" />
+    <xacro:property name="lidarOriginY"   value="0.30" />
+    <xacro:property name="lidarOriginZ"   value="0.30" />
     <!--
 	 The definitions for the ultrasonic rangefinders.
